File: intro.kicad_sch (KiCad schematic)
At the start: 122 parts, among them IC1 IS31FL3741A-QFLS4-TR, SW1 SW_Push, SW10 SW_Push, SW11 SW_Push, SW12 SW_Push, SW13 SW_Push, SW14 SW_Push, SW15 SW_Push, SW16 SW_Push, SW17 SW_Push, SW18 SW_Push, SW19 SW_Push, SW2 SW_Push, SW20 SW_Push, SW21 SW_Push, SW22 SW_Push, SW23 SW_Push, SW24 SW_Push, SW25 SW_Push, SW26 SW_Push, SW27 SW_Push, SW28 SW_Push, SW29 SW_Push, SW3 SW_Push, SW30 SW_Push, SW31 SW_Push, SW32 SW_Push, SW33 SW_Push, SW34 SW_Push, SW35 RotaryEncoder_Switch, SW4 SW_Push, SW5 SW_Push, SW6 SW_Push, SW7 SW_Push, SW8 SW_Push, SW9 SW_Push, U1 nice_nano

Commit message: Initial split setup
Parts:
- removed S1, S2: Choc_stab, intro:Kailh-PG1350-2u-STAB, symbol marbastlib-mx:MX_stab
- added C10, C2, C8: 0.1μF, Capacitor_SMD:C_0805_2012Metric, symbol Device:C_Small
- added C3, C9: 1μF, Capacitor_SMD:C_0805_2012Metric, symbol Device:C_Small
- added D36, D37, D38, D39, D40, D41, D42, D43, D44, D45, D46, D47, D48, D49, D50, D51, D52, D53, D54, D55, D56, D57, D58, D59, D60, D61, D62, D63, D64, D65, D66, D67, D68, D69, D70: 1N4148W, Diode_SMD:D_SOD-123, symbol Diode:1N4148W
- added IC2: IS31FL3741A-QFLS4-TR, QFN40P700X700X80-61N-D, symbol IS31FL3741A-QFLS4-TR:IS31FL3741A-QFLS4-TR
- added LED36, LED37, LED38, LED39, LED40, LED41, LED42, LED43, LED44, LED45, LED46, LED47, LED48, LED49, LED50, LED51, LED52, LED53, LED54, LED55, LED56, LED57, LED58, LED59, LED60, LED61, LED62, LED63, LED64, LED65, LED66, LED67, LED68, LED69, LEDB1, LEDB2, LEDB3: LED_RBAG, intro:FMB2020RGBAHG, symbol Device:LED_RBAG
- added R10: 10kΩ, Resistor_SMD:R_0805_2012Metric, symbol Device:R_Small_US
- added R6, R9: 100kΩ, Resistor_SMD:R_0805_2012Metric, symbol Device:R_Small_US
- added R7, R8: 2kΩ, Resistor_SMD:R_0805_2012Metric, symbol Device:R_Small_US
- added RSW2: SW_RST, Button_Switch_THT:SW_PUSH_6mm_H4.3mm, symbol Switch:SW_Push
- added SW36, SW37, SW38, SW39, SW40, SW41, SW44, SW45, SW46, SW47, SW48, SW49, SW50, SW51, SW52, SW53, SW54, SW55, SW57, SW58, SW59, SW60, SW61, SW62, SW63, SW67, SW68: SW_Push, intro:SW_choc_1u, symbol Switch:SW_Push
- added SW42, SW43, SW56, SW65, SW69: SW_Push, intro:SW_choc_1.5u, symbol Switch:SW_Push
- added SW64, SW66: SW_Push, intro:SW_choc_2u_STAB, symbol Switch:SW_Push
- added SW70: RotaryEncoder_Switch, intro:RotaryEncoder_Alps_EC11E-Switch_Vertical_H20mm_modified, symbol Device:RotaryEncoder_Switch
- added U2: nice_nano, intro:nice_nano_reduced, symbol nice_nano:nice_nano
- SW32, SW34: footprint intro:SW_choc_1u -> intro:SW_choc_Reversible_2u_STAB
- renumbered LED35 to LEDA1, LED36 to LEDA2, LED37 to LEDA3
Connections:
- net GND: now also C10.2, C2.2, C3.2, C8.2, C9.2, IC2.12 (GND_1), IC2.36 (GND_2), IC2.55 (GND_3), IC2.61 (EP), IC2.8 (ADDR), R10.1, R9.2, RSW2.1, SW70.C, U2.23 (GND), U2.3 (GND), U2.4 (GND)
- net SW35A: now also U1.6 (P0.20); no longer U1.12 (P1.06)
- net VCC: now also C10.1, C3.1, C8.1, C9.1, IC2.14 (AVCC), IC2.15 (PVCC_1), IC2.25 (PVCC_2), R6.1, R7.1, R8.1, U2.21 (VCC)
- net col1: now also SW13.1, SW20.1, SW27.1, SW34.1, SW6.1; no longer SW16.1, SW2.1, SW23.1, SW30.1, SW9.1
- net col2: now also SW12.1, SW19.1, SW26.1, SW33.1, SW5.1; no longer SW10.1, SW17.1, SW24.1, SW3.1, SW31.1
- net col4: now also SW10.1, SW17.1, SW24.1, SW3.1, SW31.1; no longer SW12.1, SW19.1, SW26.1, SW33.1, SW5.1
- net col5: now also SW16.1, SW2.1, SW23.1, SW30.1, SW9.1; no longer SW13.1, SW20.1, SW27.1, SW34.1, SW6.1
- net col0 renamed col6
- net col6: now also U1.12 (P1.06); no longer U1.6 (P0.20)
- new net: D51.2 (A), SW51.2
- new net: D43.2 (A), SW43.2
- new net: D67.2 (A), SW67.2
- new net: D44.2 (A), SW44.2
- new net: D62.2 (A), SW62.2
- new net: D37.2 (A), SW37.2
- new net: D42.2 (A), SW42.2
- new net: D41.2 (A), SW41.2
- new net: D64.2 (A), SW64.2
- new net: D49.2 (A), SW49.2
- new net: IC2.13 (ISET), R10.2
- new net: D52.2 (A), SW52.2
- new net: D45.2 (A), SW45.2
- new net: D54.2 (A), SW54.2
- new net: D63.2 (A), SW63.2
- new net: D40.2 (A), SW40.2
- new net: D36.2 (A), SW36.2
- new net: D69.2 (A), SW69.2
- new net: D57.2 (A), SW57.2
- new net: D46.2 (A), SW46.2
- new net: D58.2 (A), SW58.2
- new net: D65.2 (A), SW65.2
- new net: D55.2 (A), SW55.2
- new net: D38.2 (A), SW38.2
- new net: D60.2 (A), SW60.2
- new net: D47.2 (A), SW47.2
- new net: D39.2 (A), SW39.2
- new net: D56.2 (A), SW56.2
- new net: D59.2 (A), SW59.2
- new net: D66.2 (A), SW66.2
- new net: D53.2 (A), SW53.2
- new net: D61.2 (A), SW61.2
- new net: D48.2 (A), SW48.2
- new net: D50.2 (A), SW50.2
- new net: D68.2 (A), SW68.2
- new net R-CS1: IC2.26 (CS1), LED36.3 (A), LED50.3 (A)
- new net R-CS10: IC2.38 (CS12), LED45.3 (A), LED59.3 (A)
- new net R-CS11: IC2.37 (CS11), LED46.3 (A), LED60.3 (A)
- new net R-CS12: IC2.35 (CS10), LED47.3 (A), LED61.3 (A)
- new net R-CS13: IC2.34 (CS9), LED48.3 (A), LED62.3 (A)
- new net R-CS14: IC2.33 (CS8), LED49.3 (A), LED63.3 (A)
- new net R-CS15: IC2.44 (CS18), LED64.3 (A), LEDB1.3 (A)
- new net R-CS16: IC2.43 (CS17), LED65.3 (A), LEDB2.3 (A)
- new net R-CS17: IC2.42 (CS16), LED66.3 (A), LEDB3.3 (A)
- new net R-CS18: IC2.41 (CS15), LED67.3 (A)
- new net R-CS19: IC2.45 (CS19), LED68.3 (A)
- new net R-CS2: IC2.27 (CS2), LED37.3 (A), LED51.3 (A)
- new net R-CS20: IC2.46 (CS20), LED69.3 (A)
- new net R-CS3: IC2.28 (CS3), LED38.3 (A), LED52.3 (A)
- new net R-CS4: IC2.29 (CS4), LED39.3 (A), LED53.3 (A)
- new net R-CS5: IC2.30 (CS5), LED40.3 (A), LED54.3 (A)
- new net R-CS6: IC2.32 (CS7), LED41.3 (A), LED55.3 (A)
- new net R-CS7: IC2.31 (CS6), LED42.3 (A), LED56.3 (A)
- new net R-CS8: IC2.40 (CS14), LED43.3 (A), LED57.3 (A)
- new net R-CS9: IC2.39 (CS13), LED44.3 (A), LED58.3 (A)
- new net R-ENCA: SW70.A, U2.19 (AIN5/P0.29)
- new net R-ENCB: SW70.B, U2.18 (AIN0/P0.02)
- new net R-INTB: IC2.7 (INTB), R6.2, U2.5 (P0.17)
- new net R-RESET: RSW2.2, U2.22 (RST)
- new net R-RSW1: IC2.17 (SW2), LED50.2 (BK), LED51.2 (BK), LED52.2 (BK), LED53.2 (BK), LED54.2 (BK), LED55.2 (BK), LED56.2 (BK), LED57.2 (BK), LED58.2 (BK), LED59.2 (BK), LED60.2 (BK), LED61.2 (BK), LED62.2 (BK), LED63.2 (BK), LED64.2 (BK), LED65.2 (BK), LED66.2 (BK), LED67.2 (BK), LED68.2 (BK), LED69.2 (BK)
- new net R-RSW2: IC2.18 (SW3), LED50.4 (GK), LED51.4 (GK), LED52.4 (GK), LED53.4 (GK), LED54.4 (GK), LED55.4 (GK), LED56.4 (GK), LED57.4 (GK), LED58.4 (GK), LED59.4 (GK), LED60.4 (GK), LED61.4 (GK), LED62.4 (GK), LED63.4 (GK), LED64.4 (GK), LED65.4 (GK), LED66.4 (GK), LED67.4 (GK), LED68.4 (GK), LED69.4 (GK)
- new net R-RSW3: IC2.16 (SW1), LED50.1 (RK), LED51.1 (RK), LED52.1 (RK), LED53.1 (RK), LED54.1 (RK), LED55.1 (RK), LED56.1 (RK), LED57.1 (RK), LED58.1 (RK), LED59.1 (RK), LED60.1 (RK), LED61.1 (RK), LED62.1 (RK), LED63.1 (RK), LED64.1 (RK), LED65.1 (RK), LED66.1 (RK), LED67.1 (RK), LED68.1 (RK), LED69.1 (RK)
- new net R-RSW4: IC2.20 (SW5), LED36.2 (BK), LED37.2 (BK), LED38.2 (BK), LED39.2 (BK), LED40.2 (BK), LED41.2 (BK), LED42.2 (BK), LED43.2 (BK), LED44.2 (BK), LED45.2 (BK), LED46.2 (BK), LED47.2 (BK), LED48.2 (BK), LED49.2 (BK), LEDB1.2 (BK), LEDB2.2 (BK), LEDB3.2 (BK)
- new net R-RSW5: IC2.19 (SW4), LED36.4 (GK), LED37.4 (GK), LED38.4 (GK), LED39.4 (GK), LED40.4 (GK), LED41.4 (GK), LED42.4 (GK), LED43.4 (GK), LED44.4 (GK), LED45.4 (GK), LED46.4 (GK), LED47.4 (GK), LED48.4 (GK), LED49.4 (GK), LEDB1.4 (GK), LEDB2.4 (GK), LEDB3.4 (GK)
- new net R-RSW6: IC2.21 (SW6), LED36.1 (RK), LED37.1 (RK), LED38.1 (RK), LED39.1 (RK), LED40.1 (RK), LED41.1 (RK), LED42.1 (RK), LED43.1 (RK), LED44.1 (RK), LED45.1 (RK), LED46.1 (RK), LED47.1 (RK), LED48.1 (RK), LED49.1 (RK), LEDB1.1 (RK), LEDB2.1 (RK), LEDB3.1 (RK)
- new net R-SCL: IC2.10 (SCL), R7.2, U2.2 (RX1/P0.08)
- new net R-SDA: IC2.9 (SDA), R8.2, U2.1 (TX0/P0.06)
- new net R-SDB: C2.1, IC2.11 (SDB), R9.1, U2.20 (AIN7/P0.31)
- new net SW70A: SW36.1, SW43.1, SW50.1, SW57.1, SW70.S1, U2.6 (P0.20)
- new net SW70B: D70.2 (A), SW70.S2
- new net col10: SW39.1, SW46.1, SW53.1, SW60.1, SW66.1, U2.9 (P1.00)
- new net col11: SW40.1, SW47.1, SW54.1, SW61.1, SW67.1, U2.10 (P0.11)
- new net col12: SW41.1, SW48.1, SW55.1, SW62.1, SW68.1, U2.11 (P1.04)
- new net col13: SW42.1, SW49.1, SW56.1, SW63.1, SW69.1, U2.12 (P1.06)
- new net col8: SW37.1, SW44.1, SW51.1, SW58.1, SW64.1, U2.7 (P0.22)
- new net col9: SW38.1, SW45.1, SW52.1, SW59.1, SW65.1, U2.8 (P0.24)
- new net row5: D36.1 (K), D37.1 (K), D38.1 (K), D39.1 (K), D40.1 (K), D41.1 (K), D42.1 (K), U2.13 (NFC1/P0.09)
- new net row6: D43.1 (K), D44.1 (K), D45.1 (K), D46.1 (K), D47.1 (K), D48.1 (K), D49.1 (K), U2.14 (NFC2/P0.10)
- new net row7: D50.1 (K), D51.1 (K), D52.1 (K), D53.1 (K), D54.1 (K), D55.1 (K), D56.1 (K), U2.15 (P1.11)
- new net row8: D57.1 (K), D58.1 (K), D59.1 (K), D60.1 (K), D61.1 (K), D62.1 (K), D63.1 (K), U2.16 (P1.13)
- new net row9: D64.1 (K), D65.1 (K), D66.1 (K), D67.1 (K), D68.1 (K), D69.1 (K), D70.1 (K), U2.17 (P1.15)
- no-connect marks 25 -> 50
Other:
- note added: "Intro MK1"
- moved on the sheet: C1, C4, C5, C6, C7, D1, D10, D11, D12, D13, D14, D15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

Commit message: Horizontal routing start
Parts:
- SW32, SW34: footprint intro:SW_choc_Reversible_2u_STAB -> intro:SW_choc_2u_STAB
Changed lines of the file:
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@@
     (property "Reference" "SW34" (id 0) (at 353.06 257.81 0))
     (property "Value" "SW_Push" (id 1) (at 353.06 260.35 0))
-    (property "Footprint" "intro:SW_choc_Reversible_2u_STAB" (id 2) (at 353.06 260.35 0)
+    (property "Footprint" "intro:SW_choc_2u_STAB" (id 2) (at 353.06 260.35 0)
       (effects (font (size 1.27 1.27)) hide)
     )
@@
     (property "Reference" "SW32" (id 0) (at 320.04 257.81 0))
     (property "Value" "SW_Push" (id 1) (at 320.04 260.35 0))
-    (property "Footprint" "intro:SW_choc_Reversible_2u_STAB" (id 2) (at 320.04 260.35 0)
+    (property "Footprint" "intro:SW_choc_2u_STAB" (id 2) (at 320.04 260.35 0)
       (effects (font (size 1.27 1.27)) hide)
     )
@@
     )
     (path "/925bed86-c55a-4065-a929-b38a8b6f0254"
-      (reference "SW32") (unit 1) (value "SW_Push") (footprint "intro:SW_choc_Reversible_2u_STAB")
+      (reference "SW32") (unit 1) (value "SW_Push") (footprint "intro:SW_choc_2u_STAB")
     )
     (path "/60341cc5-8bc1-4a06-a6b1-f92e4d2ddecc"
@@
     )
     (path "/33096a52-edee-4914-9c26-077d40e07d9d"
-      (reference "SW34") (unit 1) (value "SW_Push") (footprint "intro:SW_choc_Reversible_2u_STAB")
+      (reference "SW34") (unit 1) (value "SW_Push") (footprint "intro:SW_choc_2u_STAB")
     )
     (path "/ed5637ea-644f-49cf-80ea-63efc66aa558"
